Commit message: latest code

File: ros2_ws_simon/src/mailrover_urdf/urdf/mail_rover.urdf.xacro (robot description, xacro)
@@ -2,8 +2,17 @@
 <robot xmlns:xacro="http://www.ros.org/wiki/xacro" name="mail_rover">
     <xacro:property name="total_mass" value="22.0"/>
-    <xacro:property name="chassis_length" value="0.40"/>
-    <xacro:property name="chassis_width" value="0.40"/>
-    <xacro:property name="chassis_height" value="0.65"/> <xacro:property name="wheel_radius" value="0.075"/> <xacro:property name="wheel_thickness" value="0.05"/>
-    <xacro:property name="wheel_mass" value="1.0"/> <xacro:property name="wheel_offset_x" value="0.15"/> <xacro:property name="wheel_offset_y" value="0.22"/> <xacro:property name="wheel_offset_z" value="0.0"/>  <material name="blue"><color rgba="0.1 0.1 0.8 1.0"/></material>
+    <xacro:property name="chassis_length" value="0.4572"/>
+    <xacro:property name="chassis_width" value="0.6096"/>
+    <xacro:property name="chassis_height" value="0.6477"/>
+    <xacro:property name="wheel_radius" value="0.0635"/>
+    <xacro:property name="wheel_thickness" value="0.05"/>
+    <xacro:property name="wheel_mass" value="1.0"/>
+    <xacro:property name="front_wheel_offset_x" value="0.27"/>
+    <xacro:property name="wheel_offset_y" value="0.2286"/>
+    <xacro:property name="rear_caster_offset_x" value="-0.18"/>
+    <xacro:property name="rear_caster_offset_y" value="0.22"/>
+    <xacro:property name="caster_radius" value="0.035"/>
+    <xacro:property name="laser_height" value="0.10"/>
+    <material name="blue"><color rgba="0.1 0.1 0.8 1.0"/></material>
     <xacro:property name="pi" value="3.141592653589793"/>
     <material name="black"><color rgba="0.1 0.1 0.1 1.0"/></material>
@@ -35,5 +44,5 @@
             <geometry><box size="${chassis_length} ${chassis_width} ${chassis_height}"/></geometry>
         </collision>
-        <xacro:box_inertia m="${total_mass - (4 * wheel_mass)}" l="${chassis_length}" w="${chassis_width}" h="${chassis_height}" xyz="0 0 0.15"/>
+        <xacro:box_inertia m="${total_mass - (2 * wheel_mass)}" l="${chassis_length}" w="${chassis_width}" h="${chassis_height}" xyz="0 0 0.15"/>
     </link>
     <joint name="base_joint" type="fixed">
@@ -58,12 +67,28 @@
             <parent link="base_link"/>
             <child link="${prefix}_wheel"/>
-            <origin xyz="${x_reflect*wheel_offset_x} ${y_reflect*wheel_offset_y} 0" rpy="0 0 0"/>
+            <origin xyz="${x_reflect*front_wheel_offset_x} ${y_reflect*wheel_offset_y} 0" rpy="0 0 0"/>
             <axis xyz="0 1 0"/>
+        </joint>
+    </xacro:macro>
+    <xacro:macro name="caster" params="prefix x_reflect y_reflect">
+        <link name="${prefix}_caster">
+            <visual>
+                <geometry><sphere radius="${caster_radius}"/></geometry>
+                <material name="black"/>
+            </visual>
+            <collision>
+                <geometry><sphere radius="${caster_radius}"/></geometry>
+            </collision>
+        </link>
+        <joint name="${prefix}_caster_joint" type="fixed">
+            <parent link="base_link"/>
+            <child link="${prefix}_caster"/>
+            <origin xyz="${x_reflect*rear_caster_offset_x} ${y_reflect*rear_caster_offset_y} ${caster_radius - wheel_radius}" rpy="0 0 0"/>
         </joint>
     </xacro:macro>
     <xacro:wheel prefix="front_left"  x_reflect="1"  y_reflect="1" />
     <xacro:wheel prefix="front_right" x_reflect="1"  y_reflect="-1" />
-    <xacro:wheel prefix="rear_left"   x_reflect="-1" y_reflect="1" />
-    <xacro:wheel prefix="rear_right"  x_reflect="-1" y_reflect="-1" />
+    <xacro:caster prefix="rear_left"  x_reflect="1" y_reflect="1" />
+    <xacro:caster prefix="rear_right" x_reflect="1" y_reflect="-1" />
     <link name="laser">
         <visual>
@@ -83,5 +108,5 @@
         <parent link="base_link"/>
         <child link="laser"/>
-        <origin xyz="0 0 ${chassis_height}" rpy="0 0 0"/>
+        <origin xyz="0 0 ${laser_height}" rpy="0 0 0"/>
     </joint>
     <gazebo reference="laser">
@@ -115,11 +140,9 @@
   <gazebo>
     <plugin name="skid_steer_drive" filename="libgazebo_ros_diff_drive.so">
-      <num_wheel_pairs>2</num_wheel_pairs>
+      <num_wheel_pairs>1</num_wheel_pairs>
       <left_joint>front_left_wheel_joint</left_joint>
       <right_joint>front_right_wheel_joint</right_joint>
-      <left_joint>rear_left_wheel_joint</left_joint>
-      <right_joint>rear_right_wheel_joint</right_joint>
-      <wheel_separation>0.44</wheel_separation>
-      <wheel_diameter>0.15</wheel_diameter>
+      <wheel_separation>0.4572</wheel_separation>
+      <wheel_diameter>0.127</wheel_diameter>
       <max_wheel_torque>20</max_wheel_torque>
       <max_wheel_acceleration>1.0</max_wheel_acceleration>

Commit message: Project backup

File: ros2_ws_simon/src/mailrover_urdf/urdf/mail_rover.urdf.xacro (robot description, xacro)
@@ -13,5 +13,5 @@
     <xacro:property name="rear_caster_offset_y" value="0.22"/>
     <xacro:property name="caster_radius" value="0.035"/>
-    <xacro:property name="laser_height" value="0.10"/>
+    <xacro:property name="laser_height" value="0.105"/>
     <material name="blue"><color rgba="0.1 0.1 0.8 1.0"/></material>
     <xacro:property name="pi" value="3.141592653589793"/>
@@ -108,5 +108,5 @@
         <parent link="base_link"/>
         <child link="laser"/>
-        <origin xyz="0 0 ${laser_height}" rpy="0 0 0"/>
+        <origin xyz="0 0 0.030" rpy="0 0 0"/>
     </joint>
     <gazebo reference="laser">
